File: PCB Design/sensor_circuit_board/sensor_circuit_board_esp32_quad/sensor_circuit_board_esp32_quad.kicad_sch (KiCad schematic)
At the start: 21 parts, among them U1 TL074, U2 TL074, U3 ESP32-DevKitC

Commit message: System identification and new PCB
Parts:
- BT1, BT2: footprint (none) -> Battery:BatteryHolder_Eagle_12BH611-GR
- R1, R10, R11, R12, R2, R3, R4, R5, R6, R7, R8, R9: footprint (none) -> Resistor_THT:R_Axial_DIN0207_L6.3mm_D2.5mm_P7.62mm_Horizontal
- Rs1, Rs2, Rs3, Rs4: footprint (none) -> Diode_THT:D_DO-15_P2.54mm_Vertical_AnodeUp
- U1, U2: footprint (none) -> Package_DIP:DIP-14_W7.62mm_LongPads
Connections:
- net at BT1.2 (-), BT2.1 (+), U1.10 (+)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: now also U3.14 (GND), U3.38 (GND)
Changed lines of the file:
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@@
   (junction (at 120.65 25.4) (diameter 0) (color 0 0 0 0)
   )
+  (junction (at 62.23 96.52) (diameter 0) (color 0 0 0 0)
+  )
   (junction (at 78.74 41.91) (diameter 0) (color 0 0 0 0)
   )
@@
   (junction (at 95.25 49.53) (diameter 0) (color 0 0 0 0)
   )
+  (junction (at 132.08 179.07) (diameter 0) (color 0 0 0 0)
+  )
   (junction (at 165.1 25.4) (diameter 0) (color 0 0 0 0)
   )
@@
     (stroke (width 0) (type default))
   )
+  (wire (pts (xy 147.32 170.18) (xy 147.32 179.07))
+    (stroke (width 0) (type default))
+  )
   (wire (pts (xy 227.33 69.85) (xy 227.33 62.23))
     (stroke (width 0) (type default))
@@
     (stroke (width 0) (type default))
   )
+  (wire (pts (xy 147.32 179.07) (xy 132.08 179.07))
+    (stroke (width 0) (type default))
+  )
   (wire (pts (xy 208.28 78.74) (xy 208.28 69.85))
     (stroke (width 0) (type default))
@@
     (stroke (width 0) (type default))
   )
-  (wire (pts (xy 62.23 25.4) (xy 62.23 105.41))
+  (wire (pts (xy 62.23 25.4) (xy 62.23 96.52))
     (stroke (width 0) (type default))
   )
@@
     (stroke (width 0) (type default))
   )
+  (wire (pts (xy 114.3 101.6) (xy 114.3 96.52))
+    (stroke (width 0) (type default))
+  )
   (wire (pts (xy 132.08 76.2) (xy 166.37 76.2))
     (stroke (width 0) (type default))
@@
     (stroke (width 0) (type default))
   )
+  (wire (pts (xy 62.23 96.52) (xy 62.23 105.41))
+    (stroke (width 0) (type default))
+  )
   (wire (pts (xy 147.32 101.6) (xy 267.97 101.6))
     (stroke (width 0) (type default))
@@
   )
   (wire (pts (xy 161.29 41.91) (xy 163.83 41.91))
+    (stroke (width 0) (type default))
+  )
+  (wire (pts (xy 114.3 96.52) (xy 62.23 96.52))
     (stroke (width 0) (type default))
   )
@@
       (effects (font (size 1.27 1.27)))
     )
-    (property "Footprint" "" (at 109.22 58.42 0)
+    (property "Footprint" "Package_DIP:DIP-14_W7.62mm_LongPads" (at 109.22 58.42 0)
       (effects (font (size 1.27 1.27)) hide)
     )
@@
       (effects (font (size 1.27 1.27)) (justify left))
     )
-    (property "Footprint" "" (at 49.53 114.046 90)
+    (property "Footprint" "Battery:BatteryHolder_Eagle_12BH611-GR" (at 49.53 114.046 90)
       (effects (font (size 1.27 1.27)) hide)
     )
@@
       (effects (font (size 1.27 1.27)))
     )
-    (property "Footprint" "" (at 172.72 51.308 90)
+    (property "Footprint" "Resistor_THT:R_Axial_DIN0207_L6.3mm_D2.5mm_P7.62mm_Horizontal" (at 172.72 51.308 90)
       (effects (font (size 1.27 1.27)) hide)
     )
@@
       (effects (font (size 1.27 1.27)))
     )
-    (property "Footprint" "" (at 213.36 51.308 90)
+    (property "Footprint" "Resistor_THT:R_Axial_DIN0207_L6.3mm_D2.5mm_P7.62mm_Horizontal" (at 213.36 51.308 90)
       (effects (font (size 1.27 1.27)) hide)
     )
@@
       (effects (font (size 1.27 1.27)) (justify right))
     )
-    (property "Footprint" "" (at 182.118 55.88 90)
+    (property "Footprint" "Diode_THT:D_DO-15_P2.54mm_Vertical_AnodeUp" (at 182.118 55.88 90)
       (effects (font (size 1.27 1.27)) hide)
     )
@@
       (effects (font (size 1.27 1.27)))
     )
-    (property "Footprint" "" (at 194.31 57.15 0)
+    (property "Footprint" "Package_DIP:DIP-14_W7.62mm_LongPads" (at 194.31 57.15 0)
       (effects (font (size 1.27 1.27)) hide)
     )
@@
       (effects (font (size 1.27 1.27)) (justify left))
     )
-    (property "Footprint" "" (at 36.83 102.87 0)
+    (property "Footprint" "Package_DIP:DIP-14_W7.62mm_LongPads" (at 36.83 102.87 0)
       (effects (font (size 1.27 1.27)) hide)
     )
@@
       (effects (font (size 1.27 1.27)) (justify left))
     )
-    (property "Footprint" "" (at 49.53 94.996 90)
+    (property "Footprint" "Battery:BatteryHolder_Eagle_12BH611-GR" (at 49.53 94.996 90)
       (effects (font (size 1.27 1.27)) hide)
     )
@@
       (effects (font (size 1.27 1.27)))
     )
-    (property "Footprint" "" (at 236.22 71.628 90)
+    (property "Footprint" "Resistor_THT:R_Axial_DIN0207_L6.3mm_D2.5mm_P7.62mm_Horizontal" (at 236.22 71.628 90)
       (effects (font (size 1.27 1.27)) hide)
     )
@@
       (effects (font (size 1.27 1.27)) (justify right))
     )
-    (property "Footprint" "" (at 137.668 55.88 90)
+    (property "Footprint" "Diode_THT:D_DO-15_P2.54mm_Vertical_AnodeUp" (at 137.668 55.88 90)
       (effects (font (size 1.27 1.27)) hide)
     )
@@
       (effects (font (size 1.27 1.27)))
     )
-    (property "Footprint" "" (at 171.45 36.83 0)
+    (property "Footprint" "Package_DIP:DIP-14_W7.62mm_LongPads" (at 171.45 36.83 0)
       (effects (font (size 1.27 1.27)) hide)
     )
@@
       (effects (font (size 1.27 1.27)))
     )
-    (property "Footprint" "" (at 195.58 71.628 90)
+    (property "Footprint" "Resistor_THT:R_Axial_DIN0207_L6.3mm_D2.5mm_P7.62mm_Horizontal" (at 195.58 71.628 90)
       (effects (font (size 1.27 1.27)) hide)
     )
@@
       (effects (font (size 1.27 1.27)))
     )
-    (property "Footprint" "" (at 152.4 57.15 0)
+    (property "Footprint" "Package_DIP:DIP-14_W7.62mm_LongPads" (at 152.4 57.15 0)
       (effects (font (size 1.27 1.27)) hide)
     )
@@
       (effects (font (size 1.27 1.27)) (justify right))
     )
-    (property "Footprint" "" (at 222.758 55.88 90)
+    (property "Footprint" "Diode_THT:D_DO-15_P2.54mm_Vertical_AnodeUp" (at 222.758 55.88 90)
       (effects (font (size 1.27 1.27)) hide)
     )
@@
       (effects (font (size 1.27 1.27)))
     )
-    (property "Footprint" "" (at 86.36 36.83 0)
+    (property "Footprint" "Package_DIP:DIP-14_W7.62mm_LongPads" (at 86.36 36.83 0)
       (effects (font (size 1.27 1.27)) hide)
     )
@@
       (effects (font (size 1.27 1.27)))
     )
-    (property "Footprint" "" (at 234.95 57.15 0)
+    (property "Footprint" "Package_DIP:DIP-14_W7.62mm_LongPads" (at 234.95 57.15 0)
       (effects (font (size 1.27 1.27)) hide)
     )
@@
       (effects (font (size 1.27 1.27)))
     )
-    (property "Footprint" "" (at 157.48 43.688 90)
+    (property "Footprint" "Resistor_THT:R_Axial_DIN0207_L6.3mm_D2.5mm_P7.62mm_Horizontal" (at 157.48 43.688 90)
       (effects (font (size 1.27 1.27)) hide)
     )
@@
       (effects (font (size 1.27 1.27)))
     )
-    (property "Footprint" "" (at 154.94 72.898 90)
+    (property "Footprint" "Resistor_THT:R_Axial_DIN0207_L6.3mm_D2.5mm_P7.62mm_Horizontal" (at 154.94 72.898 90)
       (effects (font (size 1.27 1.27)) hide)
     )
@@
       (effects (font (size 1.27 1.27)))
     )
-    (property "Footprint" "" (at 72.39 43.688 90)
+    (property "Footprint" "Resistor_THT:R_Axial_DIN0207_L6.3mm_D2.5mm_P7.62mm_Horizontal" (at 72.39 43.688 90)
       (effects (font (size 1.27 1.27)) hide)
     )
@@
       (effects (font (size 1.27 1.27)))
     )
-    (property "Footprint" "" (at 110.49 72.898 90)
+    (property "Footprint" "Resistor_THT:R_Axial_DIN0207_L6.3mm_D2.5mm_P7.62mm_Horizontal" (at 110.49 72.898 90)
       (effects (font (size 1.27 1.27)) hide)
     )
@@
       (effects (font (size 1.27 1.27)))
     )
-    (property "Footprint" "" (at 127 36.83 0)
+    (property "Footprint" "Package_DIP:DIP-14_W7.62mm_LongPads" (at 127 36.83 0)
       (effects (font (size 1.27 1.27)) hide)
     )
@@
       (effects (font (size 1.27 1.27)))
     )
-    (property "Footprint" "" (at 128.27 51.308 90)
+    (property "Footprint" "Resistor_THT:R_Axial_DIN0207_L6.3mm_D2.5mm_P7.62mm_Horizontal" (at 128.27 51.308 90)
       (effects (font (size 1.27 1.27)) hide)
     )
@@
       (effects (font (size 1.27 1.27)))
     )
-    (property "Footprint" "" (at 198.12 43.688 90)
+    (property "Footprint" "Resistor_THT:R_Axial_DIN0207_L6.3mm_D2.5mm_P7.62mm_Horizontal" (at 198.12 43.688 90)
       (effects (font (size 1.27 1.27)) hide)
     )
@@
       (effects (font (size 1.27 1.27)))
     )
-    (property "Footprint" "" (at 212.09 36.83 0)
+    (property "Footprint" "Package_DIP:DIP-14_W7.62mm_LongPads" (at 212.09 36.83 0)
       (effects (font (size 1.27 1.27)) hide)
     )
@@
       (effects (font (size 1.27 1.27)) (justify left))
     )
-    (property "Footprint" "" (at 26.67 102.87 0)
+    (property "Footprint" "Package_DIP:DIP-14_W7.62mm_LongPads" (at 26.67 102.87 0)
       (effects (font (size 1.27 1.27)) hide)
     )
@@
       (effects (font (size 1.27 1.27)))
     )
-    (property "Footprint" "" (at 87.63 51.308 90)
+    (property "Footprint" "Resistor_THT:R_Axial_DIN0207_L6.3mm_D2.5mm_P7.62mm_Horizontal" (at 87.63 51.308 90)
       (effects (font (size 1.27 1.27)) hide)
     )
@@
       (effects (font (size 1.27 1.27)) (justify right))
     )
-    (property "Footprint" "" (at 97.028 55.88 90)
+    (property "Footprint" "Diode_THT:D_DO-15_P2.54mm_Vertical_AnodeUp" (at 97.028 55.88 90)
       (effects (font (size 1.27 1.27)) hide)
     )
@@
       (effects (font (size 1.27 1.27)))
     )
-    (property "Footprint" "" (at 113.03 43.688 90)
-      (effects (font (size 1.27 1.27)) hide)
-    )
+    (property "Footprint" "Resistor_THT:R_Axial_DIN0207_L6.3mm_D2.5mm_P7.62mm_Horizontal" (at 113.03 43.688 90)
+      (effects (font (size 1.27 1.27)) hide)
+    )
