File: electronics/electronics/electronics.kicad_sch (KiCad schematic)
At the start: 21 parts, among them U1 TL071, U2 TL071, U3 TL071, U4 TL071

Commit message: Fixing rebase(hopefully)?
Parts:
- U1, U2, U3, U4: footprint (none) -> Package_DIP:DIP-14_W7.62mm_LongPads; symbol Amplifier_Operational:TL071 -> Amplifier_Operational:TL074
Connections:
- net Earth: no longer U1.4 (V-), U2.4 (V-), U3.4 (V-), U4.4 (V-)
- net at U1.1: now also R1.2, TTGO1.4 (GPIO26)
- net at BT1.1 (+): no longer U1.7 (V+)
- net at R6.2, TTGO1.6 (GPIO33): now also U3.1; no longer U3.6
- net at U4.1: now also R8.2, TTGO1.7 (GPIO32)
- net at BT4.1 (+): no longer U4.7 (V+)
- net at BT3.1 (+): no longer U3.7 (V+)
- net at BT2.1 (+): no longer U2.7 (V+)
- net at R4.2, TTGO1.5 (GPIO25): now also U2.1; no longer U2.6

Commit message: kicad update
Parts:
- removed U4: TL071, Package_DIP:DIP-14_W7.62mm_LongPads, symbol Amplifier_Operational:TL074
- added unit 5 of U1
- added unit 5 of U2
- added unit 5 of U3
- added U5: TL074, Package_DIP:DIP-14_W7.62mm_LongPads, symbol Amplifier_Operational:TL074
- U1, U2, U3: value TL071 -> TL074
Connections:
- net Earth: now also U1.11 (V-), U2.11 (V-), U3.11 (V-), U5.11 (V-), U5.3 (+)
- net at R1.2, TTGO1.4 (GPIO26): now also U5.1; no longer U1.1
- net at R2.1, R9.2: now also U5.2 (-); no longer U1.2 (-)
- net at R11.2, R5.1: now also U2.2 (-); no longer U3.2 (-)
- net at R12.2, R7.1: now also U3.2 (-)
- net at R6.2, TTGO1.6 (GPIO33): now also U2.1; no longer U3.1
- net at R8.2, TTGO1.7 (GPIO32): now also U3.1
- net at BT3.1 (+): now also U2.4 (V+)
- net at BT2.1 (+): now also U1.4 (V+)
- net at R4.2, TTGO1.5 (GPIO25): now also U1.1; no longer U2.1
- net at R10.2, R3.1: now also U1.2 (-); no longer U2.2 (-)
- net at BT1.1 (+): now also U5.4 (V+)
- net at BT4.1 (+): now also U3.4 (V+)
